File: circuit/MMMM Bottom.brd (EAGLE design)
At the start: 99.3 x 99.3 mm, 40 parts, among them J4 IN1, J9 POWER_JACKPTH_BREAD

Commit message: Updated
Parts:
- added JP25: CENTER, TOF:1X01_SIDE_NAME_SML
- added JP26: BARREL, TOF:1X01_SIDE_NAME_SML
- added JP27: GND, TOF:1X01_SIDE_NAME_SML
- added JP28: V+, TOF:1X01_SIDE_NAME_SML
- BAT_9V_+: value KEYSTONE-629+ -> KEYSTONE-637; device kanflo:KEYSTONE_BATTAERY_TERMINAL-629+ -> kanflo:KEYSTONE_AA_AAA_BATTERY_TERMINAL-637
- moved PWR1 84.9 mm to (92.1, 91.4)
- moved R2 80.5 mm to (92.1, 84.5), turned to 270 degrees
- moved J9 1.27 mm to (85.1, 99.1)
- moved BAT_9V_GND 0.64 mm to (51.4, 35.6)
Connections:
- new net N$18: J9.PWR, JP25.1
- new net N$19: J9.GND, JP26.1
- net GND: now also JP27.1; no longer J9.GND
- net N$15: now also JP28.1; no longer J9.PWR
- net N$16: now also BAT_9V_+.VCC@1, BAT_9V_+.VCC@2, BAT_9V_+.VCC@3; no longer BAT_9V_+.V+@1, BAT_9V_+.V+@2, BAT_9V_+.V+@3
Routing:
- net V+: track 246.0 -> 190.6 mm, vias 1 -> 2
- net N$15: track 11.6 -> 50.3 mm
- net N$16: track 91.7 -> 126.1 mm, vias 2 -> 0
- net N$19: track 0.00 -> 27.6 mm
- net N$18: track 0.00 -> 24.3 mm
- net N$8: track 109.6 -> 98.2 mm
- net N$12: track 92.9 -> 84.5 mm, vias 1 -> 0
- net N$4: track 41.2 -> 46.0 mm
- net N$17: track 9.78 -> 4.99 mm
- net N$9: track 107.8 -> 105.2 mm, vias 1 -> 0
- net N$43: track 101.7 -> 103.4 mm, vias 1 -> 0
- net N$10: track 93.3 -> 92.2 mm
- net N$27: track 88.4 -> 89.2 mm
- net N$1: track 4.59 -> 5.12 mm
- net N$6: track 31.5 -> 31.7 mm, vias 0 -> 1
- added copper zone on layer 1, net V+
Other:
- board text added: "MMMM BOTTOM 2018-07-05 TOFSTUFF.COM"
- board text removed: "JACKS 4x4 V0.2 FLIPPED TOFSTOFF.COM"
