File: circuit/MMMM Top.brd (EAGLE design)
At the start: 99.3 x 99.3 mm, 77 parts

Commit message: Updated
Parts:
- IC_SIG_1_2, IC_SIG_3_4, IC_SUM_1_2, IC_SUM_3_4: value TL072P -> NE5532N
Connections:
- net N$20 renamed SUM1
Other:
- board text added: "+"
- board text added: "-"
Changed lines of the file:
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@@
 <?xml version="1.0" encoding="utf-8"?>
 <!DOCTYPE eagle SYSTEM "eagle.dtd">
-<eagle version="8.6.0">
+<eagle version="9.1.1">
 <drawing>
 <settings>
@@
 <wire x1="99.314" y1="99.314" x2="99.314" y2="0" width="0" layer="20"/>
 <wire x1="99.314" y1="0" x2="0" y2="0" width="0" layer="20"/>
+<text x="74.295" y="21.59" size="1.778" layer="27">-</text>
+<text x="79.375" y="20.955" size="1.778" layer="27">+</text>
+<wire x1="73.66" y1="26.67" x2="73.66" y2="36.83" width="0.1524" layer="21"/>
+<wire x1="73.66" y1="36.83" x2="81.28" y2="36.83" width="0.1524" layer="21"/>
+<wire x1="81.28" y1="36.83" x2="81.28" y2="26.67" width="0.1524" layer="21"/>
 </plain>
 <attributes>
@@
 <param name="checkStop" value="0"/>
 <param name="checkValues" value="0"/>
+<param name="checkNames" value="1"/>
+<param name="checkWireStubs" value="1"/>
+<param name="checkPolygonWidth" value="0"/>
 <param name="useDiameter" value="13"/>
 <param name="maxErrors" value="50"/>
@@
 <element name="C1" library="adafruit" package="C025-030X050" value="1uF" x="85.725" y="23.495"/>
 <element name="C2" library="adafruit" package="C050-075X075" value="220uF" x="77.47" y="23.495" rot="R180"/>
-<element name="IC_SIG_1_2" library="linear" library_urn="urn:adsk.eagle:library:262" package="DIL08" package3d_urn="urn:adsk.eagle:package:16409/2" value="TL072P" x="61.595" y="48.26"/>
+<element name="IC_SIG_1_2" library="linear" library_urn="urn:adsk.eagle:library:262" package="DIL08" package3d_urn="urn:adsk.eagle:package:16409/2" value="NE5532N" x="61.595" y="48.26"/>
 <element name="R_IN_1" library="adafruit" package="0204/5" value="100k" x="54.61" y="48.26" rot="R90"/>
 <element name="R_BUF_1" library="adafruit" package="0204/5" value="100k" x="52.07" y="48.26" rot="R90"/>
@@
 <element name="R_BUF_2" library="adafruit" package="0204/5" value="100k" x="68.58" y="48.26" rot="R90"/>
 <element name="C_IN2" library="adafruit" package="C025-025X050" value="10uF" x="50.165" y="23.495"/>
-<element name="IC_SIG_3_4" library="linear" library_urn="urn:adsk.eagle:library:262" package="DIL08" package3d_urn="urn:adsk.eagle:package:16409/2" value="TL072P" x="86.995" y="48.26"/>
+<element name="IC_SIG_3_4" library="linear" library_urn="urn:adsk.eagle:library:262" package="DIL08" package3d_urn="urn:adsk.eagle:package:16409/2" value="NE5532N" x="86.995" y="48.26"/>
 <element name="R_IN_3" library="adafruit" package="0204/5" value="100k" x="77.47" y="48.26" rot="R270"/>
 <element name="R_BUF_3" library="adafruit" package="0204/5" value="100k" x="80.01" y="48.26" rot="R90"/>
@@
 <element name="R_BUF_4" library="adafruit" package="0204/5" value="100k" x="96.52" y="48.26" rot="R90"/>
 <element name="C_IN4" library="adafruit" package="C025-025X050" value="10uF" x="66.675" y="23.495"/>
-<element name="IC_SUM_1_2" library="linear" library_urn="urn:adsk.eagle:library:262" package="DIL08" package3d_urn="urn:adsk.eagle:package:16409/2" value="TL072P" x="13.97" y="48.26"/>
+<element name="IC_SUM_1_2" library="linear" library_urn="urn:adsk.eagle:library:262" package="DIL08" package3d_urn="urn:adsk.eagle:package:16409/2" value="NE5532N" x="13.97" y="48.26"/>
 <element name="R_1X3" library="adafruit" package="0204/5" value="100k" x="17.78" y="31.115" rot="R270"/>
 <element name="P_1X3" library="SparkFun-Electromechanical" package="ALPS_POT" value="3&gt;1" x="10.795" y="36.957" smashed="yes" rot="R270">
@@
 </element>
 <element name="C_COL3" library="adafruit" package="C025-025X050" value="10uF" x="25.4" y="23.495"/>
-<element name="IC_SUM_3_4" library="linear" library_urn="urn:adsk.eagle:library:262" package="DIL08" package3d_urn="urn:adsk.eagle:package:16409/2" value="TL072P" x="36.195" y="48.26"/>
+<element name="IC_SUM_3_4" library="linear" library_urn="urn:adsk.eagle:library:262" package="DIL08" package3d_urn="urn:adsk.eagle:package:16409/2" value="NE5532N" x="36.195" y="48.26"/>
 <element name="R_3X3" library="adafruit" package="0204/5" value="100k" x="70.485" y="31.115" rot="R270"/>
 <element name="P_3X3" library="SparkFun-Electromechanical" package="ALPS_POT" value="3&gt;3" x="63.119" y="36.957" smashed="yes" rot="R270">
@@
 <wire x1="10.6299" y1="30.1752" x2="10.795" y2="29.957" width="0.4318" layer="16"/>
 </signal>
-<signal name="N$20">
+<signal name="SUM1">
 <contactref element="P_1X4" pad="P$3"/>
 <contactref element="P_1X3" pad="P$3"/>
@@
 </signal>
 </signals>
+<mfgpreviewcolors>
+<mfgpreviewcolor name="soldermaskcolor" color="0xC8008000"/>
+<mfgpreviewcolor name="silkscreencolor" color="0xFFFEFEFE"/>
+<mfgpreviewcolor name="backgroundcolor" color="0xFF282828"/>
+<mfgpreviewcolor name="coppercolor" color="0xFFFFBF00"/>
+<mfgpreviewcolor name="substratecolor" color="0xFF786E46"/>
+</mfgpreviewcolors>
 </board>
 </drawing>
