File: circuit/MMMM Top.sch (EAGLE design)
At the start: 77 parts

Commit message: Updated
Parts:
- IC_SIG_1_2, IC_SIG_3_4, IC_SUM_1_2, IC_SUM_3_4: value TL072P -> NE5532N; device linear:TL072P -> linear:NE5532N
Connections:
- net N$20 renamed SUM1
